Commit message: Add Isaac campaign orchestration and metrics

File: description/manipulator.urdf.xacro (robot description, xacro)
@@ -1,4 +1,6 @@
 <?xml version="1.0" encoding="utf-8"?>
 <robot xmlns:xacro="http://www.ros.org/wiki/xacro" name="panda">
+  <xacro:arg name="base_xyz" default="0 0 0" />
+  <xacro:arg name="base_rpy" default="0 0 0" />
   <!-- Empty link to referr everything to -->
   <link name="world" />
@@ -7,5 +9,5 @@
   <xacro:include filename="$(find chess_manipulator)/description/panda_hand.xacro" />
   <!-- call the arm macro-->
-  <xacro:panda_arm />
+  <xacro:panda_arm base_xyz="$(arg base_xyz)" base_rpy="$(arg base_rpy)" />
   <!-- call the hand macro-->
   <xacro:panda_hand ns="panda" rpy="0 0 ${-pi/4}" connected_to="panda_link8" />

File: description/panda_arm.xacro (robot description, xacro)
@@ -42,5 +42,5 @@
   </xacro:macro>
   <xacro:macro name="panda_arm"
-    params="arm_id:='panda' description_pkg:='chess_manipulator' connected_to:='' xyz:='0 0 0' rpy:='0 0 0'">
+    params="arm_id:='panda' description_pkg:='chess_manipulator' connected_to:='' xyz:='0 0 0' rpy:='0 0 0' base_xyz:='0 0 0' base_rpy:='0 0 0'">
     <xacro:unless value="${not connected_to}">
       <joint name="${arm_id}_joint_${connected_to}" type="fixed">
@@ -55,5 +55,5 @@
       <parent link="world" />
       <child link="${arm_id}_link0" />
-      <origin xyz="0.0 0.0 0.0" rpy="0.0 0.0 0.0" />
+      <origin xyz="${base_xyz}" rpy="${base_rpy}" />
       <dynamics damping="${joint_damping}" />
     </joint>
@@ -61,10 +61,10 @@
       <visual>
         <geometry>
-          <mesh filename="file://$(find chess_manipulator)/meshes/visual/link0.dae" />
-        </geometry>
-      </visual>
-      <collision>
-        <geometry>
-          <mesh filename="file://$(find chess_manipulator)/meshes/collision/link0.stl" />
+          <mesh filename="package://chess_manipulator/meshes/visual/link0.dae" />
+        </geometry>
+      </visual>
+      <collision>
+        <geometry>
+          <mesh filename="package://chess_manipulator/meshes/collision/link0.stl" />
         </geometry>
       </collision>
@@ -78,10 +78,10 @@
       <visual>
         <geometry>
-          <mesh filename="file://$(find chess_manipulator)/meshes/visual/link1.dae" />
-        </geometry>
-      </visual>
-      <collision>
-        <geometry>
-          <mesh filename="file://$(find chess_manipulator)/meshes/collision/link1.stl" />
+          <mesh filename="package://chess_manipulator/meshes/visual/link1.dae" />
+        </geometry>
+      </visual>
+      <collision>
+        <geometry>
+          <mesh filename="package://chess_manipulator/meshes/collision/link1.stl" />
         </geometry>
       </collision>
@@ -107,10 +107,10 @@
       <visual>
         <geometry>
-          <mesh filename="file://$(find chess_manipulator)/meshes/visual/link2.dae" />
-        </geometry>
-      </visual>
-      <collision>
-        <geometry>
-          <mesh filename="file://$(find chess_manipulator)/meshes/collision/link2.stl" />
+          <mesh filename="package://chess_manipulator/meshes/visual/link2.dae" />
+        </geometry>
+      </visual>
+      <collision>
+        <geometry>
+          <mesh filename="package://chess_manipulator/meshes/collision/link2.stl" />
         </geometry>
       </collision>
@@ -136,10 +136,10 @@
       <visual>
         <geometry>
-          <mesh filename="file://$(find chess_manipulator)/meshes/visual/link3.dae" />
-        </geometry>
-      </visual>
-      <collision>
-        <geometry>
-          <mesh filename="file://$(find chess_manipulator)/meshes/collision/link3.stl" />
+          <mesh filename="package://chess_manipulator/meshes/visual/link3.dae" />
+        </geometry>
+      </visual>
+      <collision>
+        <geometry>
+          <mesh filename="package://chess_manipulator/meshes/collision/link3.stl" />
         </geometry>
       </collision>
@@ -147,5 +147,5 @@
         <origin xyz="${link3_cog}" rpy="0 0 0" />
         <mass value="${mass_link3}" />
-        <inertia ixx="0.00716" ixy="-0.00102" ixz="-0.02040" iyy="0.00920" iyz="-0.00102"
+        <inertia ixx="0.00716" ixy="0.0" ixz="0.0" iyy="0.00920" iyz="0.0"
           izz="0.007159" />
       </inertial>
@@ -166,10 +166,10 @@
       <visual>
         <geometry>
-          <mesh filename="file://$(find chess_manipulator)/meshes/visual/link4.dae" />
-        </geometry>
-      </visual>
-      <collision>
-        <geometry>
-          <mesh filename="file://$(find chess_manipulator)/meshes/collision/link4.stl" />
+          <mesh filename="package://chess_manipulator/meshes/visual/link4.dae" />
+        </geometry>
+      </visual>
+      <collision>
+        <geometry>
+          <mesh filename="package://chess_manipulator/meshes/collision/link4.stl" />
         </geometry>
       </collision>
@@ -196,10 +196,10 @@
       <visual>
         <geometry>
-          <mesh filename="file://$(find chess_manipulator)/meshes/visual/link5.dae" />
-        </geometry>
-      </visual>
-      <collision>
-        <geometry>
-          <mesh filename="file://$(find chess_manipulator)/meshes/collision/link5.stl" />
+          <mesh filename="package://chess_manipulator/meshes/visual/link5.dae" />
+        </geometry>
+      </visual>
+      <collision>
+        <geometry>
+          <mesh filename="package://chess_manipulator/meshes/collision/link5.stl" />
         </geometry>
       </collision>
@@ -207,5 +207,5 @@
         <origin xyz="${link5_cog}" rpy="0 0 0" />
         <mass value="${mass_link5}" />
-        <inertia ixx="0.0307" ixy="0.0" ixz="0.0" iyy="0.02761" iyz="-0.0613" izz="0.00818" />
+        <inertia ixx="0.0307" ixy="0.0" ixz="0.0" iyy="0.02761" iyz="0.0" izz="0.00818" />
       </inertial>
     </link>
@@ -225,10 +225,10 @@
       <visual>
         <geometry>
-          <mesh filename="file://$(find chess_manipulator)/meshes/visual/link6.dae" />
-        </geometry>
-      </visual>
-      <collision>
-        <geometry>
-          <mesh filename="file://$(find chess_manipulator)/meshes/collision/link6.stl" />
+          <mesh filename="package://chess_manipulator/meshes/visual/link6.dae" />
+        </geometry>
+      </visual>
+      <collision>
+        <geometry>
+          <mesh filename="package://chess_manipulator/meshes/collision/link6.stl" />
         </geometry>
       </collision>
@@ -254,10 +254,10 @@
       <visual>
         <geometry>
-          <mesh filename="file://$(find chess_manipulator)/meshes/visual/link7.dae" />
-        </geometry>
-      </visual>
-      <collision>
-        <geometry>
-          <mesh filename="file://$(find chess_manipulator)/meshes/collision/link7.stl" />
+          <mesh filename="package://chess_manipulator/meshes/visual/link7.dae" />
+        </geometry>
+      </visual>
+      <collision>
+        <geometry>
+          <mesh filename="package://chess_manipulator/meshes/collision/link7.stl" />
         </geometry>
       </collision>

File: description/panda_hand.xacro (robot description, xacro)
@@ -12,10 +12,10 @@
             <visual>
                 <geometry>
-                    <mesh filename="file://$(find chess_manipulator)/meshes/visual/hand.dae" />
+                    <mesh filename="package://chess_manipulator/meshes/visual/hand.dae" />
                 </geometry>
             </visual>
             <collision>
                 <geometry>
-                    <mesh filename="file://$(find chess_manipulator)/meshes/collision/hand.stl" />
+                    <mesh filename="package://chess_manipulator/meshes/collision/hand.stl" />
                 </geometry>
             </collision>
